File: pcb/digi-pot/digi-pot.sch (KiCad schematic (older format))
At the start: 2 parts

Commit message: o first schematic
Parts:
- added C? (x3): 100n, symbol C_Small
- added P?: CONN_01X12, knopf:FlatFlex, symbol CONN_01X12
- added P?: CONN_01X04, symbol CONN_01X04
- added P?: CONN_01X05, symbol CONN_01X05
- added P? (x2): CONN_01X03, symbol CONN_01X03
- added U?: DS1882, Housings_SSOP:TSSOP-16_4.4x5mm_Pitch0.65mm, symbol DS1882
Connections:
- net GND: now reaches U?.1 (GND)
- net GND: now also IC?.21 (GND), IC?.5 (GND), U?.2 (sw1), C?.2, C?.2, C?.2, P?.1 (P1), P?.3 (P3), P?.5 (P5), P?.8 (P8), U?.1 (GND), U?.2 (A2), U?.3 (A1), U?.5 (A0)
- net at U?.3 (sw2): now also IC?.3 ((PCINT26)PA2)
- net at U?.4 (B): now also IC?.22 ((PCINT25/ADC7)PA1)
- net at U?.5 (A): now also IC?.19 ((PCINT24/ADC6)PA0)
- net +5V: now reaches U?.6 (VDD)
- net +5V: now also IC?.4 (VCC), C?.1, P?.1 (P1), P?.4 (P4), P?.9 (P9), U?.16 (VDD)
- net at IC?.1 ((PCINT19/INT1)PD3): now also P?.10 (P10)
- net at IC?.15 ((PCINT3/MOSI)PB3): now also P?.4 (P4)
- net at IC?.16 ((PCINT4/MISO)PB4): now also P?.3 (P3)
- net at IC?.17 ((PCINT5/SCK)PB5): now also P?.2 (P2)
- net at IC?.2 ((PCINT20/T0)PD4): now also P?.11 (P11)
- net at IC?.26 ((PCINT11/ADC3)PC3): now also U?.12 (~CE)
- net at IC?.27 ((PCINT12/SDA/ADC4)PC4): now also U?.13 (SDA)
- net at IC?.28 ((PCINT13/SCL/ADC5)PC5): now also U?.14 (SCL)
- net at IC?.29 ((PCINT14/~RESET~)PC6): now also P?.5 (P5)
- net at IC?.30 ((PCINT16)PD0): now also P?.1 (P1)
- net at IC?.31 ((PCINT17)PD1): now also P?.2 (P2)
- net at IC?.32 ((PCINT18/INT0)PD2): now also P?.3 (P3)
- net IR-signal: now reaches IC?.6 ((PCINT27)PA3)
- net IR-signal: now also P?.6 (P6), P?.7 (P7)
- net at IC?.9 ((PCINT21/T1)PD5): now also P?.12 (P12)
- new net: P?.1 (P1), U?.10 (H1)
- new net: P?.2 (P2), U?.11 (W1)
- new net: P?.2 (P2), U?.6 (W0)
- new net: P?.3 (P3), U?.7 (L0)
- new net: P?.1 (P1), U?.8 (H0)
- new net: P?.3 (P3), U?.9 (L1)
- new net V+: C?.1, P?.2 (P2), U?.15 (V+)
- new net V-: C?.1, P?.4 (P4), U?.4 (V-)
Other:
- moved on the sheet: U?

Commit message: o complete schematic
Parts:
- added C4: 100n, Capacitors_SMD:C_0805, symbol C_Small
- added RP1, RP2: R_PACK4, Resistors_SMD:R_Array_Convex_4x0603, symbol R_PACK4
- C1, C2, C3: renamed from C?; footprint (none) -> Capacitors_SMD:C_0805
- IC1: renamed from IC?; footprint QFN/MLF32 -> Housings_DFN_QFN:QFN-32-1EP_5x5mm_Pitch0.5mm
- P1: renamed from P?; footprint (none) -> Pin_Headers:Pin_Header_Straight_1x04
- P2: renamed from P?; footprint (none) -> Pin_Headers:Pin_Header_Straight_1x05
- P3: renamed from P?; footprint knopf:FlatFlex -> knopf:FlatFlexConn
- P4, P5: renamed from P?; footprint (none) -> Pin_Headers:Pin_Header_Straight_1x03
- gave numbers to parts that had none: 2
Connections:
- net +5V: now also C4.1
- net GND: now also C4.2
- net IR-signal: now also IC1.1 ((PCINT19/INT1)PD3); no longer IC1.6 ((PCINT27)PA3)
- net Button: now reaches IC1.3 ((PCINT26)PA2), U1.3 (sw2)
- net at IC1.22 ((PCINT25/ADC7)PA1): no longer U1.4 (B)
- net at IC1.19 ((PCINT24/ADC6)PA0): no longer U1.5 (A)
- net D: now reaches P3.10 (P10)
- net D: now also RP2.2 (P2); no longer IC1.1 ((PCINT19/INT1)PD3)
- net at IC1.10 ((PCINT22/AIN0)PD6): now also RP2.6 (R3)
- net at IC1.11 ((PCINT23/AIN1)PD7): now also RP2.5 (R4)
- net MOSI: now reaches IC1.15 ((PCINT3/MOSI)PB3), P2.4 (P4)
- net MISO: now reaches IC1.16 ((PCINT4/MISO)PB4), P2.3 (P3)
- net SCK: now reaches IC1.17 ((PCINT5/SCK)PB5), P2.2 (P2)
- net at IC1.2 ((PCINT20/T0)PD4): no longer P3.11 (P11)
- net CE: now reaches IC1.26 ((PCINT11/ADC3)PC3), U2.12 (~CE)
- net SDA: now reaches IC1.27 ((PCINT12/SDA/ADC4)PC4), U2.13 (SDA)
- net SCL: now reaches IC1.28 ((PCINT13/SCL/ADC5)PC5), U2.14 (SCL)
- net RESET: now reaches IC1.29 ((PCINT14/~RESET~)PC6), P2.5 (P5)
- net at IC1.30 ((PCINT16)PD0): now also RP1.8 (R1); no longer P3.1 (P1)
- net at IC1.31 ((PCINT17)PD1): now also RP1.7 (R2); no longer P3.2 (P2)
- net at IC1.32 ((PCINT18/INT0)PD2): now also RP1.6 (R3); no longer P3.3 (P3)
- net QuadA: now reaches IC1.7 ((PCINT6/CLKI)PB6)
- net QuadA: now also U1.4 (B)
- net QuadB: now reaches IC1.8 ((PCINT7)PB7)
- net QuadB: now also U1.5 (A)
- net at IC1.9 ((PCINT21/T1)PD5): now also RP2.7 (R2); no longer P3.12 (P12)
- net Pot1_H: now reaches U2.10 (H1)
- net Pot1_H: now also P5.3 (P3); no longer P5.1 (P1)
- net Pot1_W: now reaches P5.2 (P2), U2.11 (W1)
- net Pot0_W: now reaches P4.2 (P2), U2.6 (W0)
- net Pot0_H: now reaches P4.3 (P3)
- net Pot0_H: now also U2.8 (H0); no longer U2.7 (L0)
- net Pot0_L: now reaches P4.1 (P1)
- net Pot0_L: now also U2.7 (L0); no longer U2.8 (H0)
- net Pot1_L: now reaches U2.9 (L1)
- net Pot1_L: now also P5.1 (P1); no longer P5.3 (P3)
- new net A: P3.1 (P1), RP1.1 (P1)
- new net B: P3.2 (P2), RP1.2 (P2)
- new net C: P3.3 (P3), RP1.3 (P3)
- new net E: P3.11 (P11), RP2.3 (P3)
- new net F: P3.12 (P12), RP2.4 (P4)
Other:
- moved on the sheet: P2, U1

Commit message: o Add pull-ups for I2C bus. o smallish changes in power supply.
Parts:
- added R1, R2: 4k7, Resistors_SMD:R_0603, symbol R
- C1, C2, C3, C4: footprint Capacitors_SMD:C_0805 -> Resistors_SMD:R_0603
Connections:
- net +5V: now also R1.1, R2.1
- net SCL: now also R2.2
- net SDA: now also R1.2
Changed lines of the file:
@@
 $EndComp
 $Comp
-L GND #PWR11
+L GND #PWR01
 U 1 1 580D30AA
 P 4000 1650
-F 0 "#PWR11" H 4000 1400 50  0001 C CNN
+F 0 "#PWR01" H 4000 1400 50  0001 C CNN
 F 1 "GND" H 4005 1477 50  0000 C CNN
 F 2 "" H 4000 1650 50  0000 C CNN
@@
 $EndComp
 $Comp
-L GND #PWR12
+L GND #PWR02
 U 1 1 580D3213
 P 4750 4400
-F 0 "#PWR12" H 4750 4150 50  0001 C CNN
+F 0 "#PWR02" H 4750 4150 50  0001 C CNN
 F 1 "GND" H 4755 4227 50  0000 C CNN
 F 2 "" H 4750 4400 50  0000 C CNN
@@
 V-
 $Comp
-L GND #PWR9
+L GND #PWR03
 U 1 1 580D3459
 P 2050 5500
-F 0 "#PWR9" H 2050 5250 50  0001 C CNN
+F 0 "#PWR03" H 2050 5250 50  0001 C CNN
 F 1 "GND" H 2055 5327 50  0000 C CNN
 F 2 "" H 2050 5500 50  0000 C CNN
@@
 $EndComp
 $Comp
-L +5V #PWR7
+L +5V #PWR04
 U 1 1 580D34EA
 P 1650 5300
-F 0 "#PWR7" H 1650 5150 50  0001 C CNN
+F 0 "#PWR04" H 1650 5150 50  0001 C CNN
 F 1 "+5V" H 1665 5473 50  0000 C CNN
 F 2 "" H 1650 5300 50  0000 C CNN
@@
 $EndComp
 $Comp
-L +5V #PWR3
+L +5V #PWR05
 U 1 1 580D350A
 P 1250 1850
-F 0 "#PWR3" H 1250 1700 50  0001 C CNN
+F 0 "#PWR05" H 1250 1700 50  0001 C CNN
 F 1 "+5V" H 1265 2023 50  0000 C CNN
 F 2 "" H 1250 1850 50  0000 C CNN
@@
 $EndComp
 $Comp
-L +5V #PWR16
+L +5V #PWR06
 U 1 1 580D352A
 P 5800 2500
-F 0 "#PWR16" H 5800 2350 50  0001 C CNN
+F 0 "#PWR06" H 5800 2350 50  0001 C CNN
 F 1 "+5V" H 5815 2673 50  0000 C CNN
 F 2 "" H 5800 2500 50  0000 C CNN
@@
 $EndComp
 $Comp
-L GND #PWR17
+L GND #PWR07
 U 1 1 580D354E
 P 5800 3000
-F 0 "#PWR17" H 5800 2750 50  0001 C CNN
+F 0 "#PWR07" H 5800 2750 50  0001 C CNN
 F 1 "GND" H 5805 2827 50  0000 C CNN
 F 2 "" H 5800 3000 50  0000 C CNN
@@
 $EndComp
 $Comp
-L GND #PWR4
+L GND #PWR08
 U 1 1 580D357F
 P 1250 4800
-F 0 "#PWR4" H 1250 4550 50  0001 C CNN
+F 0 "#PWR08" H 1250 4550 50  0001 C CNN
 F 1 "GND" H 1255 4627 50  0000 C CNN
 F 2 "" H 1250 4800 50  0000 C CNN
@@
 $EndComp
 $Comp
-L +5V #PWR13
+L +5V #PWR09
 U 1 1 580D36AB
 P 4850 3350
-F 0 "#PWR13" H 4850 3200 50  0001 C CNN
+F 0 "#PWR09" H 4850 3200 50  0001 C CNN
 F 1 "+5V" H 4865 3523 50  0000 C CNN
 F 2 "" H 4850 3350 50  0000 C CNN
@@
 F 0 "C1" H 1542 6196 50  0000 L CNN
 F 1 "100n" H 1542 6105 50  0000 L CNN
-F 2 "Capacitors_SMD:C_0805" H 1450 6150 50  0001 C CNN
+F 2 "Resistors_SMD:R_0603" H 1450 6150 50  0001 C CNN
 F 3 "" H 1450 6150 50  0000 C CNN
 	1    1450 6150
@@
 F 0 "C2" H 2042 6196 50  0000 L CNN
 F 1 "100n" H 2042 6105 50  0000 L CNN
-F 2 "Capacitors_SMD:C_0805" H 1950 6150 50  0001 C CNN
+F 2 "Resistors_SMD:R_0603" H 1950 6150 50  0001 C CNN
 F 3 "" H 1950 6150 50  0000 C CNN
 	1    1950 6150
@@
 $EndComp
 $Comp
-L GND #PWR6
+L GND #PWR010
 U 1 1 580D39CA
 P 1450 6250
-F 0 "#PWR6" H 1450 6000 50  0001 C CNN
+F 0 "#PWR010" H 1450 6000 50  0001 C CNN
 F 1 "GND" H 1455 6077 50  0000 C CNN
 F 2 "" H 1450 6250 50  0000 C CNN
@@
 $EndComp
 $Comp
-L GND #PWR8
+L GND #PWR011
 U 1 1 580D39ED
 P 1950 6250
-F 0 "#PWR8" H 1950 6000 50  0001 C CNN
+F 0 "#PWR011" H 1950 6000 50  0001 C CNN
 F 1 "GND" H 1955 6077 50  0000 C CNN
 F 2 "" H 1950 6250 50  0000 C CNN
@@
 $EndComp
 $Comp
-L +5V #PWR5
+L +5V #PWR012
 U 1 1 580D3A32
 P 1450 6050
-F 0 "#PWR5" H 1450 5900 50  0001 C CNN
+F 0 "#PWR012" H 1450 5900 50  0001 C CNN
 F 1 "+5V" H 1465 6223 50  0000 C CNN
 F 2 "" H 1450 6050 50  0000 C CNN
@@
 F 0 "C3" H 2442 6196 50  0000 L CNN
 F 1 "100n" H 2442 6105 50  0000 L CNN
-F 2 "Capacitors_SMD:C_0805" H 2350 6150 50  0001 C CNN
+F 2 "Resistors_SMD:R_0603" H 2350 6150 50  0001 C CNN
 F 3 "" H 2350 6150 50  0000 C CNN
 	1    2350 6150
@@
 $EndComp
 $Comp
-L GND #PWR10
+L GND #PWR013
 U 1 1 580D3AC0
 P 2350 6250
-F 0 "#PWR10" H 2350 6000 50  0001 C CNN
+F 0 "#PWR013" H 2350 6000 50  0001 C CNN
 F 1 "GND" H 2355 6077 50  0000 C CNN
 F 2 "" H 2350 6250 50  0000 C CNN
@@
 Connection ~ 5250 5300
 $Comp
-L GND #PWR15
+L GND #PWR014
 U 1 1 580D3DD5
 P 4900 5400
-F 0 "#PWR15" H 4900 5150 50  0001 C CNN
+F 0 "#PWR014" H 4900 5150 50  0001 C CNN
 F 1 "GND" H 4905 5227 50  0000 C CNN
 F 2 "" H 4900 5400 50  0000 C CNN
@@
 Connection ~ 5150 5400
 $Comp
-L +5V #PWR14
+L +5V #PWR015
 U 1 1 580D3F0C
 P 4900 5250
-F 0 "#PWR14" H 4900 5100 50  0001 C CNN
+F 0 "#PWR015" H 4900 5100 50  0001 C CNN
 F 1 "+5V" H 4915 5423 50  0000 C CNN
 F 2 "" H 4900 5250 50  0000 C CNN
@@
 F 0 "C4" H 1142 6196 50  0000 L CNN
 F 1 "100n" H 1142 6105 50  0000 L CNN
-F 2 "Capacitors_SMD:C_0805" H 1050 6150 50  0001 C CNN
+F 2 "Resistors_SMD:R_0603" H 1050 6150 50  0001 C CNN
 F 3 "" H 1050 6150 50  0000 C CNN
 	1    1050 6150
@@
 $EndComp
 $Comp
-L GND #PWR2
+L GND #PWR016
 U 1 1 580D70ED
 P 1050 6250
-F 0 "#PWR2" H 1050 6000 50  0001 C CNN
+F 0 "#PWR016" H 1050 6000 50  0001 C CNN
 F 1 "GND" H 1055 6077 50  0000 C CNN
 F 2 "" H 1050 6250 50  0000 C CNN
@@
 $EndComp
 $Comp
-L +5V #PWR1
+L +5V #PWR017
 U 1 1 580D70F3
 P 1050 6050
-F 0 "#PWR1" H 1050 5900 50  0001 C CNN
+F 0 "#PWR017" H 1050 5900 50  0001 C CNN
 F 1 "+5V" H 1065 6223 50  0000 C CNN
 F 2 "" H 1050 6050 50  0000 C CNN
@@
 	1    0    0    -1
 $EndComp
+$Comp
+L R R1
+U 1 1 581FCC3F
+P 4250 3350
+F 0 "R1" H 4100 3400 50  0000 L CNN
+F 1 "4k7" V 4250 3300 50  0000 L CNN
+F 2 "Resistors_SMD:R_0603" V 4180 3350 50  0001 C CNN
+F 3 "" H 4250 3350 50  0000 C CNN
+	1    4250 3350
+	1    0    0    -1
+$EndComp
+$Comp
+L R R2
+U 1 1 581FCCBA
+P 4450 3350
+F 0 "R2" H 4520 3396 50  0000 L CNN
+F 1 "4k7" V 4450 3300 50  0000 L CNN
+F 2 "Resistors_SMD:R_0603" V 4380 3350 50  0001 C CNN
+F 3 "" H 4450 3350 50  0000 C CNN
+	1    4450 3350
+	1    0    0    -1
+$EndComp
+Wire Wire Line
+	4450 3500 4450 3650
+Connection ~ 4450 3650
+Wire Wire Line
+	4250 3200 4700 3200
+Wire Wire Line
+	4700 3200 4700 3400
+Wire Wire Line
+	4700 3400 4850 3400
+Connection ~ 4450 3200
+Connection ~ 4850 3400
+Wire Wire Line
+	4250 3500 4250 3550
+Connection ~ 4250 3550
 $EndSCHEMATC

Commit message: o connect flat flex connector ground to ground.
Parts:
- removed P3: CONN_01X12, knopf:FlatFlexConn, symbol CONN_01X12
- added P3: CONN_01X13, knopf:FlatFlexConn, symbol CONN_01X13
Connections:
- net +5V: now also P3.4 (P4), P3.9 (P9)
- net A: now also P3.1 (P1)
- net B: now also P3.2 (P2)
- net C: now also P3.3 (P3)
- net D: now also P3.10 (P10)
- net E: now also P3.11 (P11)
- net F: now also P3.12 (P12)
- net GND: now also P3.13 (P13), P3.5 (P5), P3.8 (P8)
- net IR-signal: now also P3.6 (P6), P3.7 (P7)
Changed lines of the file:
@@
-$EndComp
-$Comp
-L CONN_01X12 P3
-U 1 1 580D2D2C
-P 5450 5350
-F 0 "P3" H 5527 5436 50  0000 L CNN
-F 1 "CONN_01X12" H 5527 5345 50  0000 L CNN
-F 2 "knopf:FlatFlexConn" H 5527 5254 50  0000 L CNN
-F 3 "" H 5450 5350 50  0000 C CNN
-	1    5450 5350
-	1    0    0    -1
 $EndComp
 $Comp
@@
 	4250 3500 4250 3550
 Connection ~ 4250 3550
+$Comp
+L CONN_01X13 P3
+U 1 1 58308878
+P 5450 5400
+F 0 "P3" H 5527 5486 50  0000 L CNN
+F 1 "CONN_01X13" H 5527 5395 50  0000 L CNN
+F 2 "knopf:FlatFlexConn" H 5527 5304 50  0000 L CNN
+F 3 "" H 5450 5400 50  0000 C CNN
+	1    5450 5400
+	1    0    0    -1
+$EndComp
+$Comp
+L GND #PWR018
+U 1 1 58308A3E
+P 5250 6050
+F 0 "#PWR018" H 5250 5800 50  0001 C CNN
+F 1 "GND" H 5255 5877 50  0000 C CNN
+F 2 "" H 5250 6050 50  0000 C CNN
+F 3 "" H 5250 6050 50  0000 C CNN
+	1    5250 6050
+	1    0    0    -1
+$EndComp
+Wire Wire Line
+	5250 6000 5250 6050
 $EndSCHEMATC
