File: pcb/remote-control/remote-control.kicad_pcb (KiCad board)
At the start: 2 copper layers, 20 x 20 mm, 13 parts, among them IC1 ATTINY44-S, P1 Bat+, P3 Bat-, Q1 Q_NMOS_GSD, T1 TEST

Commit message: o Update remote control: ready for a larger battery and housing o start housing.
Parts:
- removed R2: 1M, Resistors_SMD:R_0603
- added P2: Bat-, Pin_Headers:Pin_Header_Straight_1x01, F.Cu at (100.1, 40.4)
- Q1: value Q_NMOS_GSD -> MTM232270
- R1: value 1M -> 4R7; footprint Resistors_SMD:R_0603 -> Resistors_SMD:R_0805
- R3: value R -> 4R7
- moved R1 16.7 mm to (91.4, 54.9), turned to 315 degrees
- moved D2 5.04 mm to (92.5, 46.2), turned to 180 degrees
- moved D1 2.78 mm to (107.4, 46.0), turned to 0 degrees
- moved P3 1.02 mm to (100.1, 60.5)
- moved R3 0.96 mm to (93.2, 53.1)
Connections:
- R1 pad 1: /A -> /LEDPower
- R1 pad 2: /MOSI -> Net-(Q1-Pad3)
Routing:
- net /LED-connect: track 26.3 -> 0.00 mm
- net /LEDPower: track 2.62 -> 9.16 mm
- net /IROUT: track 6.55 -> 12.4 mm
- net VCC: track 11.3 -> 15.4 mm
- net Net-(Q1-Pad3): track 1.52 -> 4.90 mm
- net /A: track 9.56 -> 6.31 mm
- net /B: track 10.7 -> 7.73 mm
- net GND: track 36.5 -> 38.5 mm
- net /MISO: track 1.71 -> 0.00 mm
- net /MOSI: track 1.66 -> 0.02 mm
Other:
- board size 20 x 20 mm -> 26 x 26 mm
