File: pcb/remote-control/remote-control.sch (KiCad schematic (older format))
At the start: 14 parts, among them IC1 ATTINY44-S, P1 Bat+, P3 Bat-, P4 Prog, Q1 Q_NMOS_GSD, T1 TEST

Commit message: o Make IR engergy storage 1206 SMD size o add 0603 package for 100n bypass.
Parts:
- C1: value 10u -> 22u; footprint Capacitors_SMD:C_0805 -> Capacitors_SMD:C_1206
- C2: footprint (none) -> Capacitors_SMD:C_0603
Changed lines of the file:
@@
 P 1800 3250
 F 0 "C1" H 1600 3350 50  0000 L CNN
-F 1 "10u" H 1600 3150 50  0000 L CNN
-F 2 "Capacitors_SMD:C_0805" H 1838 3100 50  0001 C CNN
+F 1 "22u" H 1600 3150 50  0000 L CNN
+F 2 "Capacitors_SMD:C_1206" H 1838 3100 50  0001 C CNN
 F 3 "" H 1800 3250 50  0000 C CNN
 	1    1800 3250
@@
 F 0 "C2" H 2215 3296 50  0000 L CNN
 F 1 "100n" H 2215 3205 50  0000 L CNN
-F 2 "" H 2215 3159 50  0001 L CNN
+F 2 "Capacitors_SMD:C_0603" H 2215 3159 50  0001 L CNN
 F 3 "" H 2100 3250 50  0000 C CNN
 	1    2100 3250

Commit message: o Add some basic READMEs for the PCB directories.
Parts:
- Q1: value Q_NMOS_GSD -> MTM232270
- R3: value R -> 4R7
Changed lines of the file:
@@
 P 4450 1750
 F 0 "R3" H 4520 1796 50  0000 L CNN
-F 1 "R" H 4520 1705 50  0000 L CNN
+F 1 "4R7" H 4520 1705 50  0000 L CNN
 F 2 "Resistors_SMD:R_0805" V 4380 1750 50  0001 C CNN
 F 3 "" H 4450 1750 50  0000 C CNN
@@
 P 4600 1950
 F 0 "Q1" H 4791 1996 50  0000 L CNN
-F 1 "Q_NMOS_GSD" H 4791 1905 50  0000 L CNN
+F 1 "MTM232270" H 4791 1905 50  0000 L CNN
 F 2 "TO_SOT_Packages_SMD:SOT-323" H 4800 2050 50  0001 C CNN
 F 3 "" H 4600 1950 50  0000 C CNN
@@
 	5250 3350 4750 3350
 Wire Wire Line
-	5400 2600 5400 2650
-Connection ~ 5400 2650
-Wire Wire Line
 	4600 1750 4700 1750

Commit message: o Update remote control: ready for a larger battery and housing o start housing.
Parts:
- removed R2: 1M, Resistors_SMD:R_0603, symbol R
- added P2: Bat-, Pin_Headers:Pin_Header_Straight_1x01, symbol CONN_01X01
- R1: value 1M -> 4R7; footprint Resistors_SMD:R_0603 -> Resistors_SMD:R_0805
Connections:
- net A: no longer R1.1
- net GND: now also P2.1 (P1)
- net LEDPower: now also R1.1
- net MOSI: no longer R1.2
- net at Q1.3 (D), R3.2: now also R1.2
Other:
- moved on the sheet: E1
Changed lines of the file:
@@
 L CONN_01X05 E1
 U 1 1 5820AD2B
-P 5700 2850
-F 0 "E1" H 5777 2891 50  0000 L CNN
-F 1 "Encoder" H 5777 2800 50  0000 L CNN
-F 2 "knopf:MechanicalEncoder" H 5700 2850 50  0001 C CNN
-F 3 "" H 5700 2850 50  0000 C CNN
-	1    5700 2850
+P 5700 2950
+F 0 "E1" H 5777 2991 50  0000 L CNN
+F 1 "Encoder" H 5777 2900 50  0000 L CNN
+F 2 "knopf:MechanicalEncoder" H 5700 2950 50  0001 C CNN
+F 3 "" H 5700 2950 50  0000 C CNN
+	1    5700 2950
 	1    0    0    -1
 $EndComp
@@
 	5150 3050 5150 4100
 $Comp
-L GND #PWR01
+L GND #PWR9
 U 1 1 5820ADE0
 P 5550 4100
-F 0 "#PWR01" H 5550 3850 50  0001 C CNN
+F 0 "#PWR9" H 5550 3850 50  0001 C CNN
 F 1 "GND" H 5555 3927 50  0000 C CNN
 F 2 "" H 5550 4100 50  0000 C CNN
@@
 $EndComp
 $Comp
-L GND #PWR02
+L GND #PWR7
 U 1 1 5820B04E
 P 1950 3400
-F 0 "#PWR02" H 1950 3150 50  0001 C CNN
+F 0 "#PWR7" H 1950 3150 50  0001 C CNN
 F 1 "GND" H 1955 3227 50  0000 C CNN
 F 2 "" H 1950 3400 50  0000 C CNN
@@
 	1800 3100 2100 3100
 $Comp
-L VCC #PWR03
+L VCC #PWR5
 U 1 1 5820B189
 P 1950 3100
-F 0 "#PWR03" H 1950 2950 50  0001 C CNN
+F 0 "#PWR5" H 1950 2950 50  0001 C CNN
 F 1 "VCC" H 1967 3273 50  0000 C CNN
 F 2 "" H 1950 3100 50  0000 C CNN
@@
 Connection ~ 1950 3100
 $Comp
-L VCC #PWR04
+L VCC #PWR3
 U 1 1 5820B428
 P 2550 2650
-F 0 "#PWR04" H 2550 2500 50  0001 C CNN
+F 0 "#PWR3" H 2550 2500 50  0001 C CNN
 F 1 "VCC" H 2567 2823 50  0000 C CNN
 F 2 "" H 2550 2650 50  0000 C CNN
@@
 Connection ~ 2550 2650
 $Comp
-L GND #PWR05
+L GND #PWR4
 U 1 1 5820B656
-P 5450 2750
-F 0 "#PWR05" H 5450 2500 50  0001 C CNN
-F 1 "GND" V 5455 2622 50  0000 R CNN
-F 2 "" H 5450 2750 50  0000 C CNN
-F 3 "" H 5450 2750 50  0000 C CNN
-	1    5450 2750
+P 5450 2850
+F 0 "#PWR4" H 5450 2600 50  0001 C CNN
+F 1 "GND" V 5450 2600 50  0000 R CNN
+F 2 "" H 5450 2850 50  0000 C CNN
+F 3 "" H 5450 2850 50  0000 C CNN
+	1    5450 2850
 	0    1    1    0
 $EndComp
 Wire Wire Line
-	5450 2750 5500 2750
-$Comp
-L GND #PWR06
+	5450 2850 5500 2850
+$Comp
+L GND #PWR6
 U 1 1 5820B6D2
-P 5500 3150
-F 0 "#PWR06" H 5500 2900 50  0001 C CNN
-F 1 "GND" H 5505 2977 50  0000 C CNN
-F 2 "" H 5500 3150 50  0000 C CNN
-F 3 "" H 5500 3150 50  0000 C CNN
-	1    5500 3150
-	1    0    0    -1
-$EndComp
-Wire Wire Line
-	5500 3050 5500 3150
+P 5500 3250
+F 0 "#PWR6" H 5500 3000 50  0001 C CNN
+F 1 "GND" H 5505 3077 50  0000 C CNN
+F 2 "" H 5500 3250 50  0000 C CNN
+F 3 "" H 5500 3250 50  0000 C CNN
+	1    5500 3250
+	1    0    0    -1
+$EndComp
+Wire Wire Line
+	5500 3150 5500 3250
 $Comp
 L LED D2
@@
 $EndComp
 $Comp
-L VCC #PWR07
+L VCC #PWR1
 U 1 1 5820B8DF
 P 3150 1700
-F 0 "#PWR07" H 3150 1550 50  0001 C CNN
+F 0 "#PWR1" H 3150 1550 50  0001 C CNN
 F 1 "VCC" H 3167 1873 50  0000 C CNN
 F 2 "" H 3150 1700 50  0000 C CNN
@@
 $EndComp
 $Comp
-L GND #PWR08
+L GND #PWR2
 U 1 1 5820BB8B
 P 4700 2150
-F 0 "#PWR08" H 4700 1900 50  0001 C CNN
+F 0 "#PWR2" H 4700 1900 50  0001 C CNN
 F 1 "GND" H 4705 1977 50  0000 C CNN
 F 2 "" H 4700 2150 50  0000 C CNN
@@
 Text Label 4400 2350 1    60   ~ 0
 IROUT
-Text Label 5300 2650 0    60   ~ 0
+Text Label 5300 2750 0    60   ~ 0
 A
-Text Label 5300 2850 0    60   ~ 0
+Text Label 5300 2950 0    60   ~ 0
 B
-Text Label 5500 2950 2    60   ~ 0
+Text Label 5500 3050 2    60   ~ 0
 Button
 $Comp
-L R R1
-U 1 1 5820C3D0
-P 5100 3250
-F 0 "R1" V 5200 3200 50  0000 L CNN
-F 1 "1M" V 5100 3200 50  0000 L CNN
-F 2 "Resistors_SMD:R_0603" V 5030 3250 50  0001 C CNN
-F 3 "" H 5100 3250 50  0000 C CNN
-	1    5100 3250
-	0    1    1    0
-$EndComp
-$Comp
-L R R2
-U 1 1 5820C452
-P 5000 2850
-F 0 "R2" V 4900 2800 50  0000 L CNN
-F 1 "1M" V 5000 2800 50  0000 L CNN
-F 2 "Resistors_SMD:R_0603" V 4930 2850 50  0001 C CNN
-F 3 "" H 5000 2850 50  0000 C CNN
-	1    5000 2850
-	0    1    1    0
-$EndComp
-$Comp
-L GND #PWR09
+L GND #PWR8
 U 1 1 5820EE3F
-P 2550 3900
-F 0 "#PWR09" H 2550 3650 50  0001 C CNN
-F 1 "GND" H 2555 3727 50  0000 C CNN
-F 2 "" H 2550 3900 50  0000 C CNN
-F 3 "" H 2550 3900 50  0000 C CNN
-	1    2550 3900
-	1    0    0    -1
-$EndComp
-Wire Wire Line
-	2550 3850 2550 3900
-Connection ~ 2550 3850
+P 2500 4000
+F 0 "#PWR8" H 2500 3750 50  0001 C CNN
+F 1 "GND" H 2505 3827 50  0000 C CNN
+F 2 "" H 2500 4000 50  0000 C CNN
+F 3 "" H 2500 4000 50  0000 C CNN
+	1    2500 4000
+	1    0    0    -1
+$EndComp
 Wire Wire Line
 	4750 3550 5300 3550
 Wire Wire Line
-	5300 3550 5300 2950
-Wire Wire Line
-	5300 2950 5500 2950
-Wire Wire Line
-	4750 2950 5150 2950
-Wire Wire Line
-	5150 2950 5150 2850
-Wire Wire Line
-	5250 2650 5500 2650
-Wire Wire Line
-	5250 2650 5250 3350
+	5300 3050 5500 3050
+Wire Wire Line
+	4750 2950 5500 2950
+Wire Wire Line
+	5250 2750 5500 2750
 Wire Wire Line
 	5250 3350 4750 3350
@@
 Wire Wire Line
 	3150 1750 3200 1750
-Connection ~ 5150 2850
 Wire Wire Line
 	3600 1750 3700 1750
 Text Label 3700 1750 1    60   ~ 0
 LED-connect
-Connection ~ 4950 3250
-Connection ~ 5250 3250
-Wire Wire Line
-	5150 2850 5500 2850
-Wire Wire Line
-	4850 2850 4850 3150
-Connection ~ 4850 3150
 Text Label 4200 1750 1    60   ~ 0
 LEDPower
 Wire Wire Line
 	4100 1750 4300 1750
+Wire Wire Line
+	5250 3350 5250 2750
+Wire Wire Line
+	5300 3550 5300 3050
+$Comp
+L R R1
+U 1 1 583237B4
+P 4450 1450
+F 0 "R1" H 4520 1496 50  0000 L CNN
+F 1 "4R7" H 4520 1405 50  0000 L CNN
+F 2 "Resistors_SMD:R_0805" V 4380 1450 50  0001 C CNN
+F 3 "" H 4450 1450 50  0000 C CNN
+	1    4450 1450
+	0    -1   -1   0
+$EndComp
+Wire Wire Line
+	4300 1750 4300 1450
+Wire Wire Line
+	4600 1450 4600 1750
+Connection ~ 4600 1750
+Connection ~ 4300 1750
+$Comp
+L CONN_01X01 P2
+U 1 1 58323947
+P 2300 4000
+F 0 "P2" H 2219 3775 50  0000 C CNN
+F 1 "Bat-" H 2219 3866 50  0000 C CNN
+F 2 "Pin_Headers:Pin_Header_Straight_1x01" H 2219 3867 50  0001 C CNN
+F 3 "" H 2300 4000 50  0000 C CNN
+	1    2300 4000
+	-1   0    0    1
+$EndComp
+Wire Wire Line
+	2500 4000 2500 3850
+Connection ~ 2500 3850
+Connection ~ 2500 4000
 $EndSCHEMATC
